File: hw/Eagle/alpha85+mem+acia+pio-routed.brd (EAGLE design)
At the start: 100 x 80 mm, 33 parts, among them IC2 74HC573N, IC3 62256, IC4 28C256, IC5 74HCT00N, IC7 74HCT245N, IC9 74HCT138N, Q1 3.6864

Commit message: Schematic revised
Connections:
- net A4: no longer IC4.5
- net A5: now also IC3.5, IC4.5
Changed lines of the file:
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@@
 <wire x1="28.0035" y1="62.1792" x2="27.94" y2="62.23" width="0.3048" layer="1"/>
 <wire x1="48.1203" y1="41.9481" x2="48.26" y2="41.91" width="0.3048" layer="1"/>
+<contactref element="IC3" pad="5"/>
+<contactref element="IC4" pad="5"/>
+<wire x1="77.47" y1="15.24" x2="96.52" y2="15.24" width="0" layer="19" extent="1-1"/>
+<wire x1="77.3811" y1="15.3162" x2="77.47" y2="15.24" width="0" layer="19" extent="16-16"/>
 </signal>
 <signal name="A4">
@@
 <contactref element="IC3" pad="6"/>
 <contactref element="IC4" pad="6"/>
-<contactref element="IC4" pad="5"/>
 <contactref element="IC9" pad="2"/>
 <wire x1="96.4692" y1="17.7165" x2="96.52" y2="17.78" width="0.3048" layer="1"/>
@@
 <wire x1="96.3549" y1="17.7165" x2="96.52" y2="17.78" width="0.3048" layer="1"/>
 <wire x1="77.6097" y1="17.8308" x2="77.47" y2="17.78" width="0.3048" layer="1"/>
-<wire x1="96.4692" y1="17.7165" x2="96.52" y2="15.24" width="0" layer="19" extent="1-1"/>
 </signal>
 <signal name="A3">
