File: hw/Eagle/alpha85+mem+acia+pio-routed.sch (EAGLE design)
At the start: 33 parts, among them IC2 74HC573N, IC3 62256, IC4 28C256, IC5 74HCT00N, IC7 74HCT245N, IC9 74HCT138N, Q1 3.6864

Commit message: Schematic revised
Connections:
- net A4: no longer IC4G$1.A5
- net A5: now also IC3.A5, IC4G$1.A5
Other:
- moved on the sheet: C9, IC7, IC7P
