File: hw/Eagle/alpha-issue2-v23.brd (EAGLE design)
At the start: 100 x 83.8 mm, 37 parts, among them IC2 74HC573N, IC3 62256, IC4 28C256, IC5 74HCT00N, IC7 74HCT245N, IC9 74HCT138N, Q1 3.6864

Commit message: BRD REV
Parts:
- C1, C2: value 56 -> 33
- C12: value (none) -> 100n
- IC1: value (none) -> 80C85
- IC6: value (none) -> 68B50
- IC8: value (none) -> 82C55
- R3: value (none) -> 330
Other:
- board text added: "+5 GND"
