File: hw/Eagle/alpha-issue2-v23.sch (EAGLE design)
At the start: 37 parts, among them IC2 74HC573N, IC3 62256, IC4 28C256, IC5 74HCT00N, IC7 74HCT245N, IC9 74HCT138N, Q1 3.6864

Commit message: BRD REV
Parts:
- C1, C2: value 56 -> 33
- C12: value (none) -> 100n
- IC1: value (none) -> 80C85
- IC6: value (none) -> 68B50
- IC8: value (none) -> 82C55
- R3: value (none) -> 330
Changed lines of the file:
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@@
 </classes>
 <parts>
-<part name="IC1" library="micro-intel" deviceset="8085" device=""/>
+<part name="IC1" library="micro-intel" deviceset="8085" device="" value="80C85"/>
 <part name="IC2" library="74xx-eu" deviceset="74*573" device="N" technology="HC"/>
 <part name="Q1" library="crystal" deviceset="CRYSTAL" device="HC49S" value="3.6864"/>
-<part name="C1" library="rcl" deviceset="C-EU" device="025-040X050" value="56"/>
-<part name="C2" library="rcl" deviceset="C-EU" device="025-040X050" value="56"/>
+<part name="C1" library="rcl" deviceset="C-EU" device="025-040X050" value="33"/>
+<part name="C2" library="rcl" deviceset="C-EU" device="025-040X050" value="33"/>
 <part name="GND1" library="supply1" deviceset="GND" device=""/>
 <part name="GND2" library="supply1" deviceset="GND" device=""/>
@@
 <part name="GND9" library="supply1" deviceset="GND" device=""/>
 <part name="D2" library="Seeed-LED" library_urn="urn:adsk.eagle:library:472" deviceset="DIP-LED-GREEN-GREEN(2P-D5MM)" device="" package3d_urn="urn:adsk.eagle:package:32744/1" value="G502DC"/>
-<part name="R3" library="rcl" deviceset="R-EU_" device="0207/7"/>
+<part name="R3" library="rcl" deviceset="R-EU_" device="0207/7" value="330"/>
 <part name="GND10" library="supply1" deviceset="GND" device=""/>
 <part name="IC3" library="memory-hitachi" deviceset="62256P" device="" value="62256"/>
@@
 <part name="P+7" library="supply1" deviceset="VCC" device=""/>
 <part name="GND13" library="supply1" deviceset="GND" device=""/>
-<part name="IC6" library="micro-motorola" deviceset="6850" device=""/>
+<part name="IC6" library="micro-motorola" deviceset="6850" device="" value="68B50"/>
 <part name="GND15" library="supply1" deviceset="GND" device=""/>
 <part name="GND16" library="supply1" deviceset="GND" device=""/>
@@
 <part name="P+9" library="supply1" deviceset="VCC" device=""/>
 <part name="GND17" library="supply1" deviceset="GND" device=""/>
-<part name="IC8" library="micro-intel" deviceset="8255A" device=""/>
+<part name="IC8" library="micro-intel" deviceset="8255A" device="" value="82C55"/>
 <part name="JP2" library="pinhead" deviceset="PINHD-2X5" device=""/>
 <part name="JP3" library="pinhead" deviceset="PINHD-2X5" device=""/>
@@
 <part name="P+11" library="supply1" deviceset="VCC" device=""/>
 <part name="GND19" library="supply1" deviceset="GND" device=""/>
-<part name="C12" library="rcl" deviceset="C-EU" device="050-025X075"/>
+<part name="C12" library="rcl" deviceset="C-EU" device="050-025X075" value="100n"/>
 <part name="C8" library="rcl" deviceset="C-EU" device="050-025X075"/>
 <part name="GND20" library="supply1" deviceset="GND" device=""/>
